File: DesignFiles/122025.kicad_pcb (KiCad board)
At the start: 2 copper layers, 77 x 60 mm, 54 parts, among them J1 IN, J2 OUT, J3 PWR, J4 LED, J5 GND, Q1 2N5088, Q2 2N4401, U1 JRC4558

Commit message: Add files via upload
Parts:
- added REF**: MountingHole_3.2mm_M3, MountingHole:MountingHole_3.2mm_M3, F.Cu at (40.0, 18.0)
- added REF**: MountingHole_3.2mm_M3, MountingHole:MountingHole_3.2mm_M3, F.Cu at (18.0, 30.0)
- added REF**: MountingHole_3.2mm_M3, MountingHole:MountingHole_3.2mm_M3, F.Cu at (83.0, 16.0)
- added REF**: MountingHole_3.2mm_M3, MountingHole:MountingHole_3.2mm_M3, F.Cu at (61.0, 68.0)
Routing:
- net /LED GND: track 90.8 -> 87.0 mm
- net Net-(R4-Pad1): track 83.8 -> 81.3 mm
- net Net-(Q1-E): track 19.5 -> 17.4 mm
- net Net-(Q1-C): track 95.9 -> 96.7 mm
